File: pcb/watchwinder.brd (EAGLE design)
At the start: 160 x 100 mm, 9 parts

Commit message: Compacted a bit
Parts:
- moved ON 31.0 mm to (87.6, 63.5)
- moved PWR 31.0 mm to (87.6, 50.8)
- moved SEL2 22.5 mm to (57.1, 64.8)
- moved OMEGA 22.5 mm to (6.35, 11.4)
- moved MOTOR 22.5 mm to (26.7, 19.1)
- moved MULTIPLEXER 22.5 mm to (34.3, 61.0)
- moved ROLEX 22.5 mm to (6.35, 20.3)
- moved MCU 22.5 mm to (63.5, 25.4)
- moved SEL1 22.5 mm to (12.7, 66.0)
Routing:
- net N$15: track 143.1 -> 133.8 mm
- net N$14: track 112.7 -> 105.6 mm
Other:
- board outline removed
