File: pcb/ watchwinder mirror.brd (EAGLE design)
At the start: 9 parts

Commit message: Prepped for cnc
Parts:
- moved ROLEX 43.1 mm to (72.4, 57.1), turned to 0 degrees
- moved OMEGA 30.7 mm to (83.8, 57.1), turned to 0 degrees
- moved MOTOR 26.9 mm to (78.7, 25.4)
- moved ON 12.7 mm to (33.0, 58.4)
- moved PWR 12.7 mm to (17.8, 58.4)
- moved MCU 10.2 mm to (52.1, 24.1)
- moved SEL1 6.35 mm to (29.2, 38.1)
- moved MULTIPLEXER 6.35 mm to (15.2, 36.8)
- moved SEL2 5.24 mm to (5.08, 39.4)
Routing:
- net N$9: track 8.89 -> 35.5 mm
- net N$14: track 170.5 -> 145.7 mm
- net N$8: track 8.89 -> 32.5 mm
- net N$4: track 26.3 -> 5.45 mm
- net N$6: track 25.5 -> 5.45 mm
- net N$5: track 25.5 -> 5.45 mm
- net N$3: track 23.4 -> 5.45 mm
- net N$7: track 23.3 -> 5.45 mm
- net N$11: track 10.2 -> 27.6 mm
- net N$12: track 50.6 -> 33.6 mm
- net N$1: track 22.4 -> 7.01 mm
- net N$2: track 21.6 -> 7.01 mm
- net N$10: track 10.2 -> 23.4 mm
- net N$27: track 40.2 -> 33.2 mm
- net N$25: track 25.6 -> 19.1 mm
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